File: design/pc-amplifier/bluetooth-src.kicad_sch (KiCad schematic)
At the start: 7 parts, among them U6 MC78L05, U7 AC6939-MODULE

Commit message: Add page settings to PCB and schematic.
Other:
- company: (none) -> Dilshan R Jayakody
- title: (none) -> Arduino Mini Amplifier
Changed lines of the file:
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@@
 (kicad_sch (version 20211123) (generator eeschema)
   (paper "A4")
+  (title_block
+    (title "Arduino Mini Amplifier")
+    (date "2022-07-30")
+    (rev "1.0.0")
+    (company "Dilshan R Jayakody")
+    (comment 1 "jayakody2000lk@gmail.com")
+    (comment 2 "https://github.com/dilshan/arduino-mini-amp")
+  )
   (junction (at 147.32 123.19) (diameter 0) (color 0 0 0 0)
   )
