File: design/pc-amplifier/control-module.kicad_sch (KiCad schematic)
At the start: 15 parts, among them SW1 6mm Tactile SW, SW2 6mm Tactile SW, SW3 6mm Tactile SW, SW4 6mm Tactile SW

Commit message: Add page settings to PCB and schematic.
Other:
- company: (none) -> Dilshan R Jayakody
- title: (none) -> Arduino Mini Amplifier
Changed lines of the file:
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@@
 (kicad_sch (version 20211123) (generator eeschema)
   (paper "A4")
+  (title_block
+    (title "Arduino Mini Amplifier")
+    (date "2022-07-30")
+    (rev "1.0.0")
+    (company "Dilshan R Jayakody")
+    (comment 1 "jayakody2000lk@gmail.com")
+    (comment 2 "https://github.com/dilshan/arduino-mini-amp")
+  )
   (junction (at 236.22 77.47) (diameter 0) (color 0 0 0 0)
   )
