File: design/pc-amplifier/pc-amplifier.kicad_sch (KiCad schematic)
At the start: 13 parts, among them J1 PJ307, J2 DC-005, J3 PJ307, J4 AV-8.4-3, J5 AV-8.4-3

Commit message: Initial version of the PCB.
Parts:
- R1, R2: footprint Resistor_SMD:R_0805_2012Metric_Pad1.20x1.40mm_HandSolder -> Resistor_THT:R_Axial_DIN0204_L3.6mm_D1.6mm_P1.90mm_Vertical
Changed lines of the file:
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@@
     (property "Reference" "R1" (id 0) (at 139.7 152.4 90))
     (property "Value" "0R" (id 1) (at 139.7 154.94 90))
-    (property "Footprint" "Resistor_SMD:R_0805_2012Metric_Pad1.20x1.40mm_HandSolder" (id 2) (at 139.7 160.528 90)
+    (property "Footprint" "Resistor_THT:R_Axial_DIN0204_L3.6mm_D1.6mm_P1.90mm_Vertical" (id 2) (at 139.7 160.528 90)
       (effects (font (size 1.27 1.27)) hide)
     )
@@
     (property "Reference" "R2" (id 0) (at 139.7 163.83 90))
     (property "Value" "0R" (id 1) (at 139.7 166.37 90))
-    (property "Footprint" "Resistor_SMD:R_0805_2012Metric_Pad1.20x1.40mm_HandSolder" (id 2) (at 139.7 171.958 90)
+    (property "Footprint" "Resistor_THT:R_Axial_DIN0204_L3.6mm_D1.6mm_P1.90mm_Vertical" (id 2) (at 139.7 171.958 90)
       (effects (font (size 1.27 1.27)) hide)
     )
@@
       (reference "#PWR0148") (unit 1) (value "GNDA") (footprint "")
     )
-    (path "/362dc043-966c-4bd9-b11d-1034a60ee1a6/09ccd545-709a-49f0-bafe-6770c5abddae"
-      (reference "#PWR0149") (unit 1) (value "GNDA") (footprint "")
-    )
     (path "/362dc043-966c-4bd9-b11d-1034a60ee1a6/47b09b77-c6a5-4f4b-beab-fb015ac7544f"
       (reference "#PWR0150") (unit 1) (value "GNDD") (footprint "")
@@
       (reference "#PWR0225") (unit 1) (value "GNDA") (footprint "")
     )
+    (path "/362dc043-966c-4bd9-b11d-1034a60ee1a6/53f0f51d-9f76-4e9e-9918-88b799543560"
+      (reference "#PWR?") (unit 1) (value "GND") (footprint "")
+    )
     (path "/bbf6665a-0726-424c-8919-000ceceaec9d/c8b2177d-d956-405f-ac31-a3d3e8631cfa"
       (reference "A1") (unit 1) (value "Arduino Nano V3") (footprint "Module:Arduino_Nano")
@@
     )
     (path "/4a987034-4782-4d3d-a9b2-48b19a94c53a"
-      (reference "R1") (unit 1) (value "0R") (footprint "Resistor_SMD:R_0805_2012Metric_Pad1.20x1.40mm_HandSolder")
+      (reference "R1") (unit 1) (value "0R") (footprint "Resistor_THT:R_Axial_DIN0204_L3.6mm_D1.6mm_P1.90mm_Vertical")
     )
     (path "/e246f5e8-ec22-4141-b6b8-29cb3989af2b"
-      (reference "R2") (unit 1) (value "0R") (footprint "Resistor_SMD:R_0805_2012Metric_Pad1.20x1.40mm_HandSolder")
+      (reference "R2") (unit 1) (value "0R") (footprint "Resistor_THT:R_Axial_DIN0204_L3.6mm_D1.6mm_P1.90mm_Vertical")
     )
     (path "/3bb9c3d4-9a6f-41ac-8d1e-92ed4fe334c0/c004c559-dd72-4b0b-bd1b-2f5664fa3918"

Commit message: Routed PCB design for REV 1.0.
Parts:
- added H1, H2: 2.5mm hole, MountingHole:MountingHole_2.5mm_Pad, symbol Mechanical:MountingHole_Pad
Connections:
- net GNDA: now also H1.1, H2.1
Changed lines of the file:
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@@
+    (stroke (width 0) (type default) (color 0 0 0 0))
+  )
+  (wire (pts (xy 203.2 138.43) (xy 203.2 147.32))
     (stroke (width 0) (type default) (color 0 0 0 0))
   )
@@
     (stroke (width 0) (type default) (color 0 0 0 0))
   )
+  (wire (pts (xy 238.76 138.43) (xy 238.76 147.32))
+    (stroke (width 0) (type default) (color 0 0 0 0))
+  )
   (wire (pts (xy 64.77 172.72) (xy 64.77 176.53))
     (stroke (width 0.25) (type default) (color 0 72 0 1))
@@
   (text "SPEAKER-LEFT" (at 252.73 100.33 0)
     (effects (font (size 1.27 1.27)) (justify left bottom))
+  )
+  (symbol (lib_id "power:GNDA") (at 203.2 147.32 0) (unit 1)
+    (in_bom yes) (on_board yes) (fields_autoplaced)
+    (property "Reference" "#PWR01" (id 0) (at 203.2 153.67 0)
+      (effects (font (size 1.27 1.27)) hide)
+    )
+    (property "Value" "GNDA" (id 1) (at 203.2 152.4 0))
+    (property "Footprint" "" (id 2) (at 203.2 147.32 0)
+      (effects (font (size 1.27 1.27)) hide)
+    )
+    (property "Datasheet" "" (id 3) (at 203.2 147.32 0)
+      (effects (font (size 1.27 1.27)) hide)
+    )
+    (pin "1")
   )
   (symbol (lib_id "power:GND") (at 83.82 176.53 0) (unit 1)
@@
     (pin "1")
   )
+  (symbol (lib_id "Mechanical:MountingHole_Pad") (at 238.76 135.89 0) (unit 1)
+    (in_bom yes) (on_board yes) (fields_autoplaced)
+    (property "Reference" "H2" (id 0) (at 241.3 133.3499 0)
+      (effects (font (size 1.27 1.27)) (justify left))
+    )
+    (property "Value" "2.5mm hole" (id 1) (at 241.3 135.8899 0)
+      (effects (font (size 1.27 1.27)) (justify left))
+    )
+    (property "Footprint" "MountingHole:MountingHole_2.5mm_Pad" (id 2) (at 238.76 135.89 0)
+      (effects (font (size 1.27 1.27)) hide)
+    )
+    (property "Datasheet" "~" (id 3) (at 238.76 135.89 0)
+      (effects (font (size 1.27 1.27)) hide)
+    )
+    (pin "1")
+  )
   (symbol (lib_id "Device:Polyfuse") (at 57.15 160.02 90) (unit 1)
     (in_bom yes) (on_board yes) (fields_autoplaced)
@@
     (pin "2")
   )
+  (symbol (lib_id "Mechanical:MountingHole_Pad") (at 203.2 135.89 0) (unit 1)
+    (in_bom yes) (on_board yes) (fields_autoplaced)
+    (property "Reference" "H1" (id 0) (at 205.74 133.3499 0)
+      (effects (font (size 1.27 1.27)) (justify left))
+    )
+    (property "Value" "2.5mm hole" (id 1) (at 205.74 135.8899 0)
+      (effects (font (size 1.27 1.27)) (justify left))
+    )
+    (property "Footprint" "MountingHole:MountingHole_2.5mm_Pad" (id 2) (at 203.2 135.89 0)
+      (effects (font (size 1.27 1.27)) hide)
+    )
+    (property "Datasheet" "~" (id 3) (at 203.2 135.89 0)
+      (effects (font (size 1.27 1.27)) hide)
+    )
+    (pin "1")
+  )
   (symbol (lib_id "power:PWR_FLAG") (at 151.13 170.18 0) (unit 1)
     (in_bom yes) (on_board yes) (fields_autoplaced)
@@
     )
     (property "Datasheet" "~" (id 3) (at 83.82 154.94 0)
+      (effects (font (size 1.27 1.27)) hide)
+    )
+    (pin "1")
+  )
+  (symbol (lib_id "power:GNDA") (at 238.76 147.32 0) (unit 1)
+    (in_bom yes) (on_board yes) (fields_autoplaced)
+    (property "Reference" "#PWR02" (id 0) (at 238.76 153.67 0)
+      (effects (font (size 1.27 1.27)) hide)
+    )
+    (property "Value" "GNDA" (id 1) (at 238.76 152.4 0))
+    (property "Footprint" "" (id 2) (at 238.76 147.32 0)
+      (effects (font (size 1.27 1.27)) hide)
+    )
+    (property "Datasheet" "" (id 3) (at 238.76 147.32 0)
       (effects (font (size 1.27 1.27)) hide)
     )
@@
       (reference "#FLG0107") (unit 1) (value "PWR_FLAG") (footprint "")
     )
+    (path "/14e702f6-af6e-4971-b3c5-9682f7d557f0"
+      (reference "#PWR01") (unit 1) (value "GNDA") (footprint "")
+    )
+    (path "/d6f72c6e-1e35-4a14-b8f0-9b0eb6f35dac"
+      (reference "#PWR02") (unit 1) (value "GNDA") (footprint "")
+    )
+    (path "/362dc043-966c-4bd9-b11d-1034a60ee1a6/53f0f51d-9f76-4e9e-9918-88b799543560"
+      (reference "#PWR03") (unit 1) (value "GND") (footprint "")
+    )
     (path "/d162f4d2-fad4-48d6-974e-dde6cc1f5177"
       (reference "#PWR0101") (unit 1) (value "GNDA") (footprint "")
@@
       (reference "#PWR0225") (unit 1) (value "GNDA") (footprint "")
     )
-    (path "/362dc043-966c-4bd9-b11d-1034a60ee1a6/53f0f51d-9f76-4e9e-9918-88b799543560"
-      (reference "#PWR?") (unit 1) (value "GND") (footprint "")
-    )
     (path "/bbf6665a-0726-424c-8919-000ceceaec9d/c8b2177d-d956-405f-ac31-a3d3e8631cfa"
       (reference "A1") (unit 1) (value "Arduino Nano V3") (footprint "Module:Arduino_Nano")
@@
       (reference "F1") (unit 1) (value "RUEF300 ") (footprint "Fuse:Fuse_Bourns_MF-RHT300")
     )
+    (path "/a7f29850-1cc4-46c1-b46d-ef6833aa6812"
+      (reference "H1") (unit 1) (value "2.5mm hole") (footprint "MountingHole:MountingHole_2.5mm_Pad")
+    )
+    (path "/89e1a620-d5c2-446d-9fa9-2ea7c80a2848"
+      (reference "H2") (unit 1) (value "2.5mm hole") (footprint "MountingHole:MountingHole_2.5mm_Pad")
+    )
     (path "/2ccde68a-58ee-4378-8723-11728eb99a66"

Commit message: Add page settings to PCB and schematic.
Other:
- company: (none) -> Dilshan R Jayakody
- title: (none) -> Arduino Mini Amplifier
Changed lines of the file:
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@@
 (kicad_sch (version 20211123) (generator eeschema)
   (paper "A4")
+  (title_block
+    (title "Arduino Mini Amplifier")
+    (date "2022-07-30")
+    (rev "1.0.0")
+    (company "Dilshan R Jayakody")
+    (comment 1 "jayakody2000lk@gmail.com")
+    (comment 2 "https://github.com/dilshan/arduino-mini-amp")
+  )
   (junction (at 129.54 170.18) (diameter 0) (color 0 0 0 0)
   )
