File: design/pc-amplifier/power-amplifier.kicad_sch (KiCad schematic)
At the start: 40 parts, among them K1 HK19F-DC-12-SHG, Q1 BC858, Q2 BC817, Q3 BC817, Q4 BC817, U5 YDA138

Commit message: Initial version of the PCB.
Connections:
- net GNDA: no longer Q2.2 (E)
- new net GND: Q2.2 (E)
Changed lines of the file:
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@@
-    (pin "1")
-  )
-  (symbol (lib_id "power:GNDA") (at 85.09 184.15 0) (unit 1)
-    (in_bom yes) (on_board yes) (fields_autoplaced)
-    (property "Reference" "#PWR0149" (id 0) (at 85.09 190.5 0)
-      (effects (font (size 1.27 1.27)) hide)
-    )
-    (property "Value" "GNDA" (id 1) (at 85.09 189.23 0))
-    (property "Footprint" "" (id 2) (at 85.09 184.15 0)
-      (effects (font (size 1.27 1.27)) hide)
-    )
-    (property "Datasheet" "" (id 3) (at 85.09 184.15 0)
-      (effects (font (size 1.27 1.27)) hide)
-    )
     (pin "1")
   )
@@
       (effects (font (size 1.27 1.27)) hide)
     )
+    (pin "1")
+  )
+  (symbol (lib_id "power:GND") (at 85.09 184.15 0) (unit 1)
+    (in_bom yes) (on_board yes) (fields_autoplaced)
+    (property "Reference" "#PWR?" (id 0) (at 85.09 190.5 0)
+      (effects (font (size 1.27 1.27)) hide)
+    )
+    (property "Value" "GND" (id 1) (at 85.09 189.23 0))
+    (property "Footprint" "" (id 2) (at 85.09 184.15 0)
+      (effects (font (size 1.27 1.27)) hide)
+    )
+    (property "Datasheet" "" (id 3) (at 85.09 184.15 0)
+      (effects (font (size 1.27 1.27)) hide)
+    )

Commit message: Add page settings to PCB and schematic.
Other:
- company: (none) -> Dilshan R Jayakody
- title: (none) -> Arduino Mini Amplifier
Changed lines of the file:
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@@
 (kicad_sch (version 20211123) (generator eeschema)
   (paper "A4")
+  (title_block
+    (title "Arduino Mini Amplifier")
+    (date "2022-07-30")
+    (rev "1.0.0")
+    (company "Dilshan R Jayakody")
+    (comment 1 "jayakody2000lk@gmail.com")
+    (comment 2 "https://github.com/dilshan/arduino-mini-amp")
+  )
   (junction (at 196.85 125.095) (diameter 0) (color 0 0 0 0)
   )
